File: fan.kicad_sch (KiCad schematic)
At the start: 9 parts, among them J4 Conn_01x04, Q1 BSS138

Commit message: update schematic BOM and some part substitutions
Parts:
- C77: DK 478-KGM05AR71C104KHCT-ND -> 490-10700-1-ND; LCSC C307331 -> C77020; PARTNO KGM05AR71C104KH -> GRM155R71H104KE14D; Voltage (none) -> 50V
- R2, R34: LCSC (none) -> C25744
Changed lines of the file:
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@@
-			)
-		)
-		(property "ALT1" ""
-			(at 127 92.71 0)
-			(hide yes)
-			(show_name no)
-			(do_not_autoplace no)
-			(effects
-				(font
-					(size 1.27 1.27)
-				)
 			)
 		)
@@
 			)
 		)
-		(property "Mouser" ""
-			(at 168.91 91.44 0)
-			(hide yes)
-			(show_name no)
-			(do_not_autoplace no)
-			(effects
-				(font
-					(size 1.27 1.27)
-				)
-			)
-		)
 		(property "Manufacturer" ""
 			(at 168.91 91.44 90)
@@
 			)
 		)
-		(property "ALT1" ""
-			(at 168.91 91.44 90)
-			(hide yes)
-			(show_name no)
-			(do_not_autoplace no)
-			(effects
-				(font
-					(size 1.27 1.27)
-				)
-			)
-		)
 		(property "Sim.Device" ""
 			(at 168.91 91.44 90)
@@
 		)
 		(property "Sim.Pins" ""
+			(at 168.91 91.44 90)
+			(hide yes)
+			(show_name no)
+			(do_not_autoplace no)
+			(effects
+				(font
+					(size 1.27 1.27)
+				)
+			)
+		)
+		(property "LCSC" "C25744"
 			(at 168.91 91.44 90)
 			(hide yes)
@@
 			)
 		)
-		(property "Mouser" ""
-			(at 229.87 80.01 0)
-			(hide yes)
-			(show_name no)
-			(do_not_autoplace no)
-			(effects
-				(font
-					(size 1.27 1.27)
-				)
-			)
-		)
 		(property "Manufacturer" ""
 			(at 229.87 80.01 0)
@@
 			)
 		)
-		(property "ALT1" ""
-			(at 229.87 80.01 0)
-			(hide yes)
-			(show_name no)
-			(do_not_autoplace no)
-			(effects
-				(font
-					(size 1.27 1.27)
-				)
-			)
-		)
 		(property "Sim.Device" ""
 			(at 229.87 80.01 0)
@@
 		)
 		(property "Sim.Pins" ""
+			(at 229.87 80.01 0)
+			(hide yes)
+			(show_name no)
+			(do_not_autoplace no)
+			(effects
+				(font
+					(size 1.27 1.27)
+				)
+			)
+		)
+		(property "LCSC" "C25744"
 			(at 229.87 80.01 0)
 			(hide yes)
@@
 			)
 		)
-		(property "ALT1" ""
-			(at 175.26 99.06 90)
-			(hide yes)
-			(show_name no)
-			(do_not_autoplace no)
-			(effects
-				(font
-					(size 1.27 1.27)
-				)
-			)
-		)
 		(property "Sim.Device" ""
 			(at 175.26 99.06 90)
@@
 			)
 		)
-		(property "Mouser" ""
-			(at 250.19 92.71 0)
-			(hide yes)
-			(show_name no)
-			(do_not_autoplace no)
-			(effects
-				(font
-					(size 1.27 1.27)
-				)
-			)
-		)
 		(property "Manufacturer" ""
-			(at 250.19 92.71 0)
-			(hide yes)
-			(show_name no)
-			(do_not_autoplace no)
-			(effects
-				(font
-					(size 1.27 1.27)
-				)
-			)
-		)
-		(property "ALT1" ""
 			(at 250.19 92.71 0)
 			(hide yes)
@@
 			)
 		)
-		(property "Mouser" ""
-			(at 209.55 80.01 0)
-			(hide yes)
-			(show_name no)
-			(do_not_autoplace no)
-			(effects
-				(font
-					(size 1.27 1.27)
-				)
-			)
-		)
 		(property "Manufacturer" ""
-			(at 209.55 80.01 0)
-			(hide yes)
-			(show_name no)
-			(do_not_autoplace no)
-			(effects
-				(font
-					(size 1.27 1.27)
-				)
-			)
-		)
-		(property "ALT1" ""
 			(at 209.55 80.01 0)
 			(hide yes)
@@
 			)
 		)
-		(property "Mouser" ""
-			(at 111.76 92.71 0)
-			(hide yes)
-			(show_name no)
-			(do_not_autoplace no)
-			(effects
-				(font
-					(size 1.27 1.27)
-				)
-			)
-		)
 		(property "Manufacturer" ""
-			(at 111.76 92.71 90)
-			(hide yes)
-			(show_name no)
-			(do_not_autoplace no)
-			(effects
-				(font
-					(size 1.27 1.27)
-				)
-			)
-		)
-		(property "ALT1" ""
 			(at 111.76 92.71 90)
 			(hide yes)
@@
 			)
 		)
-		(property "PARTNO" "KGM05AR71C104KH"
+		(property "PARTNO" "GRM155R71H104KE14D"
 			(at 220.98 80.01 0)
 			(hide yes)
@@
 			)
 		)
-		(property "DK" "478-KGM05AR71C104KHCT-ND"
-			(at 220.98 80.01 0)
-			(hide yes)
-			(show_name no)
-			(do_not_autoplace no)
-			(effects
-				(font
-					(size 1.27 1.27)
-				)
-			)
-		)
-		(property "Mouser" ""
+		(property "DK" "490-10700-1-ND"
 			(at 220.98 80.01 0)
 			(hide yes)
@@
 			)
 		)
-		(property "LCSC" "C307331"
-			(at 220.98 80.01 0)
-			(hide yes)
-			(show_name no)
-			(do_not_autoplace no)
-			(effects
-				(font
-					(size 1.27 1.27)
-				)
-			)
-		)
-		(property "ALT1" ""
+		(property "LCSC" "C77020"
 			(at 220.98 80.01 0)
 			(hide yes)
@@
 		)
 		(property "Sim.Pins" ""
+			(at 220.98 80.01 0)
+			(hide yes)
+			(show_name no)
+			(do_not_autoplace no)
+			(effects
+				(font
+					(size 1.27 1.27)
+				)
+			)
+		)
+		(property "Voltage" "50V"
 			(at 220.98 80.01 0)
 			(hide yes)
@@
 			)
 		)
-		(property "Mouser" ""
-			(at 218.44 99.06 90)
-			(hide yes)
-			(show_name no)
-			(do_not_autoplace no)
-			(effects
-				(font
-					(size 1.27 1.27)
-				)
-			)
-		)
 		(property "Manufacturer" ""
 			(at 218.44 99.06 90)
 			(hide yes)
-			(show_name no)
-			(do_not_autoplace no)
-			(effects
-				(font
-					(size 1.27 1.27)
-				)
-			)
-		)
-		(property "ALT1" ""
-			(at 218.44 99.06 90)
-			(hide yes)
