File: fan.kicad_sch (KiCad schematic)
At the start: 9 parts, among them J4 Conn_01x04, Q1 BSS138

Commit message: changed fan connector footprint back to normal. lots of part substitutions for JLCPCB. Mounting hole changes for enclosure
Parts:
- C76: footprint Capacitor_SMD:C_0603_1608Metric -> Capacitor_SMD:C_1210_3225Metric; DK 490-18214-1-ND -> (none); LCSC (none) -> C138687; Manufacturer (none) -> Samsung Electro-Mechanics; PARTNO GRM188R61E106KA73D -> CL32B106KBJNNNE; Voltage 25V -> 50V
- C77: DK 490-10700-1-ND -> (none); LCSC C77020 -> C307331; Manufacturer (none) -> Samsung Electro-Mechanics; PARTNO GRM155R71H104KE14D -> CL05B104KB54PNC
- R1: DK 311-1.00KLRCT-ND -> (none); LCSC (none) -> C11702; Manufacturer (none) -> UNI-ROYAL(Uniroyal Elec); PARTNO RC0402FR-071KL -> 0402WGF1001TCE
- R2, R34: DK 311-10KJRCT-ND -> (none); Manufacturer (none) -> UNI-ROYAL(Uniroyal Elec); PARTNO RC0402JR-0710KL -> 0402WGF1002TCE
- R33: DK 311-5.6KLRCT-ND -> (none); LCSC (none) -> C25908; Manufacturer (none) -> UNI-ROYAL(Uniroyal Elec); PARTNO RC0402FR-075K6L -> 0402WGF5601TCE
Changed lines of the file:
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@@
 			)
 		)
-		(property "Datasheet" ""
+		(property "Datasheet" "https://www.lcsc.com/datasheet/lcsc_datasheet_2411221126_UNI-ROYAL-Uniroyal-Elec-0402WGF1002TCE_C25744.pdf"
 			(at 168.91 91.44 0)
 			(hide yes)
@@
 			)
 		)
-		(property "PARTNO" "RC0402JR-0710KL"
+		(property "PARTNO" "0402WGF1002TCE"
 			(at 168.91 91.44 0)
 			(hide yes)
@@
 			)
 		)
-		(property "DK" "311-10KJRCT-ND"
+		(property "DK" ""
 			(at 168.91 91.44 0)
 			(hide yes)
@@
 			)
 		)
-		(property "Manufacturer" ""
+		(property "Manufacturer" "UNI-ROYAL(Uniroyal Elec)"
 			(at 168.91 91.44 90)
 			(hide yes)
@@
 			)
 		)
-		(property "Datasheet" ""
+		(property "Datasheet" "https://www.lcsc.com/datasheet/lcsc_datasheet_2411221126_UNI-ROYAL-Uniroyal-Elec-0402WGF1002TCE_C25744.pdf"
 			(at 229.87 80.01 0)
 			(hide yes)
@@
 			)
 		)
-		(property "PARTNO" "RC0402JR-0710KL"
+		(property "PARTNO" "0402WGF1002TCE"
 			(at 229.87 80.01 0)
 			(hide yes)
@@
 			)
 		)
-		(property "DK" "311-10KJRCT-ND"
+		(property "DK" ""
 			(at 229.87 80.01 0)
 			(hide yes)
@@
 			)
 		)
-		(property "Manufacturer" ""
+		(property "Manufacturer" "UNI-ROYAL(Uniroyal Elec)"
 			(at 229.87 80.01 0)
 			(hide yes)
@@
 			)
 		)
-		(property "Datasheet" ""
+		(property "Datasheet" "https://www.lcsc.com/datasheet/lcsc_datasheet_2206010045_UNI-ROYAL-Uniroyal-Elec-0402WGF5601TCE_C25908.pdf"
 			(at 209.55 80.01 0)
 			(hide yes)
@@
 			)
 		)
-		(property "DK" "311-5.6KLRCT-ND"
+		(property "LCSC" "C25908"
 			(at 209.55 80.01 0)
 			(hide yes)
@@
 			)
 		)
-		(property "PARTNO" "RC0402FR-075K6L"
+		(property "DK" ""
 			(at 209.55 80.01 0)
 			(hide yes)
@@
 			)
 		)
-		(property "Manufacturer" ""
+		(property "PARTNO" "0402WGF5601TCE"
+			(at 209.55 80.01 0)
+			(hide yes)
+			(show_name no)
+			(do_not_autoplace no)
+			(effects
+				(font
+					(size 1.27 1.27)
+				)
+			)
+		)
+		(property "Manufacturer" "UNI-ROYAL(Uniroyal Elec)"
 			(at 209.55 80.01 0)
 			(hide yes)
@@
 			)
 		)
-		(property "Datasheet" ""
+		(property "Datasheet" "https://www.lcsc.com/datasheet/lcsc_datasheet_2206010216_UNI-ROYAL-Uniroyal-Elec-0402WGF1001TCE_C11702.pdf"
 			(at 111.76 92.71 0)
 			(hide yes)
@@
 			)
 		)
-		(property "PARTNO" "RC0402FR-071KL"
+		(property "LCSC" "C11702"
 			(at 111.76 92.71 0)
 			(hide yes)
@@
 			)
 		)
-		(property "DK" "311-1.00KLRCT-ND"
+		(property "PARTNO" "0402WGF1001TCE"
 			(at 111.76 92.71 0)
 			(hide yes)
@@
 			)
 		)
-		(property "Manufacturer" ""
+		(property "DK" ""
+			(at 111.76 92.71 0)
+			(hide yes)
+			(show_name no)
+			(do_not_autoplace no)
+			(effects
+				(font
+					(size 1.27 1.27)
+				)
+			)
+		)
+		(property "Manufacturer" "UNI-ROYAL(Uniroyal Elec)"
 			(at 111.76 92.71 90)
 			(hide yes)
@@
 			)
 		)
-		(property "Datasheet" ""
+		(property "Datasheet" "https://www.lcsc.com/datasheet/lcsc_datasheet_2304140030_Samsung-Electro-Mechanics-CL05B104KB54PNC_C307331.pdf"
 			(at 220.98 80.01 0)
 			(hide yes)
@@
 			)
 		)
-		(property "PARTNO" "GRM155R71H104KE14D"
+		(property "PARTNO" "CL05B104KB54PNC"
 			(at 220.98 80.01 0)
 			(hide yes)
@@
 			)
 		)
-		(property "DK" "490-10700-1-ND"
+		(property "DK" ""
 			(at 220.98 80.01 0)
 			(hide yes)
@@
 			)
 		)
-		(property "Manufacturer" ""
+		(property "Manufacturer" "Samsung Electro-Mechanics"
 			(at 220.98 80.01 0)
 			(hide yes)
@@
 			)
 		)
-		(property "LCSC" "C77020"
+		(property "LCSC" "C307331"
 			(at 220.98 80.01 0)
 			(hide yes)
@@
 			)
 		)
-		(property "Footprint" "Capacitor_SMD:C_0603_1608Metric"
+		(property "Footprint" "Capacitor_SMD:C_1210_3225Metric"
 			(at 218.44 99.06 0)
 			(hide yes)
@@
 			)
 		)
-		(property "Datasheet" ""
+		(property "Datasheet" "https://product.samsungsem.com/mlcc/CL32B106KBJNNN.do"
 			(at 218.44 99.06 0)
 			(hide yes)
@@
 			)
 		)
-		(property "Description" "Unpolarized capacitor, small symbol"
+		(property "Description" "10uF 50V X7R ±10% 1210 MLCC"
 			(at 218.44 99.06 0)
 			(hide yes)
@@
 			)
 		)
-		(property "Voltage" "25V"
+		(property "Voltage" "50V"
 			(at 222.504 95.25 90)
 			(show_name no)
@@
 			)
 		)
-		(property "PARTNO" "GRM188R61E106KA73D"
+		(property "PARTNO" "CL32B106KBJNNNE"
 			(at 218.44 99.06 0)
 			(hide yes)
@@
 			)
 		)
-		(property "DK" "490-18214-1-ND"
+		(property "DK" ""
 			(at 218.44 99.06 0)
 			(hide yes)
@@
 			)
 		)
-		(property "Manufacturer" ""
+		(property "Manufacturer" "Samsung Electro-Mechanics"
 			(at 218.44 99.06 90)
 			(hide yes)
@@
 			(hide yes)
 			(show_name no)
+			(do_not_autoplace no)
+			(effects
+				(font
+					(size 1.27 1.27)
+				)
+			)
+		)
+		(property "LCSC" "C138687"
+			(at 218.44 99.06 0)
+			(hide yes)
+			(show_name no)

Commit message: re-added many missing LCSC part numbers that got lost in translation
Parts:
- D13: LCSC (none) -> C24672
- Q1: LCSC (none) -> C7420339
Changed lines of the file:
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@@
 		(pin "2"
 		)
-		(instances
+		    (property "LCSC" "C7420339"
+      (at 0 0 0)
+      (effects (font (size 1.27 1.27)) (hide yes))
+    )
+    (instances
 			(project "bitaxeProto"
 				(path "/61fe8d2c-9301-4ad9-8caf-c47acfa835b0/edab3562-ad75-4c4e-afab-a1841dcf5714"
@@
 		(pin "2"
 		)
-		(instances
+		    (property "LCSC" "C24672"
+      (at 0 0 0)
+      (effects (font (size 1.27 1.27)) (hide yes))
+    )
+    (instances
 			(project "bitaxeProto"
 				(path "/61fe8d2c-9301-4ad9-8caf-c47acfa835b0/edab3562-ad75-4c4e-afab-a1841dcf5714"

Commit message: DRC fixes. added filled via notes. power track tweaking. switched fan connecter back to normal (again)
Parts:
- J4: footprint bitaxe:470531000 -> bitaxe:fan_connector
Changed lines of the file:
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@@
+			)
+		)
+		(property "LCSC" "C7420339"
+			(at 0 0 0)
+			(hide yes)
+			(show_name no)
+			(do_not_autoplace no)
+			(effects
+				(font
+					(size 1.27 1.27)
+				)
 			)
 		)
@@
 		(pin "2"
 		)
-		    (property "LCSC" "C7420339"
-      (at 0 0 0)
-      (effects (font (size 1.27 1.27)) (hide yes))
-    )
-    (instances
+		(instances
 			(project "bitaxeProto"
 				(path "/61fe8d2c-9301-4ad9-8caf-c47acfa835b0/edab3562-ad75-4c4e-afab-a1841dcf5714"
@@
 			)
 		)
+		(property "LCSC" "C24672"
+			(at 0 0 0)
+			(hide yes)
+			(show_name no)
+			(do_not_autoplace no)
+			(effects
+				(font
+					(size 1.27 1.27)
+				)
+			)
+		)
 		(pin "1"
 		)
 		(pin "2"
 		)
-		    (property "LCSC" "C24672"
-      (at 0 0 0)
-      (effects (font (size 1.27 1.27)) (hide yes))
-    )
-    (instances
+		(instances
 			(project "bitaxeProto"
 				(path "/61fe8d2c-9301-4ad9-8caf-c47acfa835b0/edab3562-ad75-4c4e-afab-a1841dcf5714"
@@
 			)
 		)
-		(property "Footprint" "bitaxe:470531000"
+		(property "Footprint" "bitaxe:fan_connector"
 			(at 250.19 92.71 0)
 			(hide yes)

Commit message: switch to cheaper USB-C connector
Parts:
- D13: DK DDZ9684-7DICT-ND -> (none); PARTNO DDZ9684-7 -> MMSZ4684T1G
- Q1: DK BSS138K-13DICT-ND -> (none); PARTNO BSS138K-13 -> BSS138
Changed lines of the file:
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@@
 			)
 		)
-		(property "PARTNO" "BSS138K-13"
+		(property "PARTNO" "BSS138"
 			(at 127 92.71 0)
 			(hide yes)
@@
 			)
 		)
-		(property "DK" "BSS138K-13DICT-ND"
+		(property "DK" ""
 			(at 127 92.71 0)
 			(hide yes)
@@
 			)
 		)
-		(property "PARTNO" "DDZ9684-7"
+		(property "PARTNO" "MMSZ4684T1G"
 			(at 175.26 99.06 0)
 			(hide yes)
@@
 			)
 		)
-		(property "DK" "DDZ9684-7DICT-ND"
+		(property "DK" ""
 			(at 175.26 99.06 0)
 			(hide yes)

Commit message: updated part attributes for JLCPCB Fabrication Toolkit
Parts:
- Q1: FT Rotation Offset (none) -> 180
Changed lines of the file:
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@@
+			)
+		)
+		(property "FT Rotation Offset" "180"
+			(at 127 92.71 0)
+			(hide yes)
+			(show_name no)
+			(do_not_autoplace no)
+			(effects
+				(font
+					(size 1.27 1.27)
+				)
 			)
 		)
