File: level_shifter.kicad_sch (KiCad schematic)
At the start: 11 parts, among them U19 TLV3542

Commit message: update schematic BOM and some part substitutions
Parts:
- C206: DK 478-KGM05AR71C104KHCT-ND -> 490-10700-1-ND; LCSC (none) -> C77020; PARTNO KGM05AR71C104KH -> GRM155R71H104KE14D; Voltage (none) -> 50V
- C207: LCSC (none) -> C52923
- R56, R57, R59, R60: LCSC (none) -> C25744
Changed lines of the file:
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@@
-			)
-		)
-		(property "ALT1" ""
-			(at 208.28 57.15 0)
-			(hide yes)
-			(show_name no)
-			(do_not_autoplace no)
-			(effects
-				(font
-					(size 1.27 1.27)
-				)
 			)
 		)
@@
 		)
 		(property "Sim.Pins" ""
+			(at 208.28 57.15 0)
+			(hide yes)
+			(show_name no)
+			(do_not_autoplace no)
+			(effects
+				(font
+					(size 1.27 1.27)
+				)
+			)
+		)
+		(property "LCSC" "C52923"
 			(at 208.28 57.15 0)
 			(hide yes)
@@
 			)
 		)
-		(property "ALT1" ""
-			(at 111.76 58.42 90)
-			(hide yes)
-			(show_name no)
-			(do_not_autoplace no)
-			(effects
-				(font
-					(size 1.27 1.27)
-				)
-			)
-		)
 		(property "Sim.Device" ""
 			(at 111.76 58.42 90)
@@
 			)
 		)
-		(property "ALT1" ""
-			(at 111.76 68.58 90)
-			(hide yes)
-			(show_name no)
-			(do_not_autoplace no)
-			(effects
-				(font
-					(size 1.27 1.27)
-				)
-			)
-		)
 		(property "Sim.Device" ""
 			(at 111.76 68.58 90)
@@
 		)
 		(property "Sim.Pins" ""
+			(at 111.76 68.58 90)
+			(hide yes)
+			(show_name no)
+			(do_not_autoplace no)
+			(effects
+				(font
+					(size 1.27 1.27)
+				)
+			)
+		)
+		(property "LCSC" "C25744"
 			(at 111.76 68.58 90)
 			(hide yes)
@@
 			)
 		)
-		(property "ALT1" ""
-			(at 129.54 91.44 0)
-			(hide yes)
-			(show_name no)
-			(do_not_autoplace no)
-			(effects
-				(font
-					(size 1.27 1.27)
-				)
-			)
-		)
 		(property "Sim.Device" ""
 			(at 129.54 91.44 0)
@@
 			)
 		)
-		(property "ALT1" ""
-			(at 111.76 88.9 90)
-			(hide yes)
-			(show_name no)
-			(do_not_autoplace no)
-			(effects
-				(font
-					(size 1.27 1.27)
-				)
-			)
-		)
 		(property "Sim.Device" ""
 			(at 111.76 88.9 90)
@@
 			)
 		)
-		(property "DK" "478-KGM05AR71C104KHCT-ND"
+		(property "DK" "490-10700-1-ND"
 			(at 201.93 57.15 0)
 			(hide yes)
@@
 			)
 		)
-		(property "PARTNO" "KGM05AR71C104KH"
-			(at 201.93 57.15 0)
-			(hide yes)
-			(show_name no)
-			(do_not_autoplace no)
-			(effects
-				(font
-					(size 1.27 1.27)
-				)
-			)
-		)
-		(property "ALT1" ""
+		(property "PARTNO" "GRM155R71H104KE14D"
 			(at 201.93 57.15 0)
 			(hide yes)
@@
 		)
 		(property "Sim.Pins" ""
+			(at 201.93 57.15 0)
+			(hide yes)
+			(show_name no)
+			(do_not_autoplace no)
+			(effects
+				(font
+					(size 1.27 1.27)
+				)
+			)
+		)
+		(property "Voltage" "50V"
+			(at 201.93 57.15 0)
+			(hide yes)
+			(show_name no)
+			(do_not_autoplace no)
+			(effects
+				(font
+					(size 1.27 1.27)
+				)
+			)
+		)
+		(property "LCSC" "C77020"
 			(at 201.93 57.15 0)
 			(hide yes)
@@
 			)
 		)
-		(property "ALT1" ""
-			(at 134.62 77.47 90)
-			(hide yes)
-			(show_name no)
-			(do_not_autoplace no)
-			(effects
-				(font
-					(size 1.27 1.27)
-				)
-			)
-		)
 		(property "Sim.Device" ""
 			(at 134.62 77.47 90)
@@
 			)
 		)
-		(property "ALT1" ""
-			(at 134.62 46.99 90)
-			(hide yes)
-			(show_name no)
-			(do_not_autoplace no)
-			(effects
-				(font
-					(size 1.27 1.27)
-				)
-			)
-		)
 		(property "Sim.Device" ""
 			(at 134.62 46.99 90)
@@
 			)
 		)
-		(property "ALT1" ""
-			(at 111.76 63.5 90)
-			(hide yes)
-			(show_name no)
-			(do_not_autoplace no)
-			(effects
-				(font
-					(size 1.27 1.27)
-				)
-			)
-		)
 		(property "Sim.Device" ""
 			(at 111.76 63.5 90)
@@
 		)
 		(property "Sim.Pins" ""
+			(at 111.76 63.5 90)
+			(hide yes)
+			(show_name no)
+			(do_not_autoplace no)
+			(effects
+				(font
+					(size 1.27 1.27)
+				)
+			)
+		)
+		(property "LCSC" "C25744"
 			(at 111.76 63.5 90)
 			(hide yes)
@@
 			)
 		)
-		(property "ALT1" ""
-			(at 129.54 60.96 0)
-			(hide yes)
-			(show_name no)
-			(do_not_autoplace no)
-			(effects
-				(font
-					(size 1.27 1.27)
-				)
-			)
-		)
 		(property "Sim.Device" ""
 			(at 129.54 60.96 0)
@@
 			)
 		)
-		(property "ALT1" ""
-			(at 111.76 99.06 90)
-			(hide yes)
-			(show_name no)
-			(do_not_autoplace no)
-			(effects
-				(font
-					(size 1.27 1.27)
-				)
-			)
-		)
 		(property "Sim.Device" ""
 			(at 111.76 99.06 90)
@@
 		)
 		(property "Sim.Pins" ""
+			(at 111.76 99.06 90)
+			(hide yes)
+			(show_name no)
+			(do_not_autoplace no)
+			(effects
+				(font
+					(size 1.27 1.27)
+				)
+			)
+		)
+		(property "LCSC" "C25744"
 			(at 111.76 99.06 90)
 			(hide yes)
@@
 			)
 		)
-		(property "ALT1" ""
-			(at 111.76 93.98 90)
-			(hide yes)
-			(show_name no)
-			(do_not_autoplace no)
-			(effects
-				(font
-					(size 1.27 1.27)
-				)
-			)
-		)
 		(property "Sim.Device" ""
 			(at 111.76 93.98 90)
@@
 			(at 111.76 93.98 90)
 			(hide yes)
+			(show_name no)
+			(do_not_autoplace no)
+			(effects
+				(font
+					(size 1.27 1.27)
+				)
+			)
+		)
+		(property "LCSC" "C25744"
+			(at 111.76 93.98 90)
+			(hide yes)

Commit message: update U19 footprint for #1. fix TP silkscreen orientation
Parts:
- U19: footprint Package_SO:SOIC-8_5.3x5.3mm_P1.27mm -> bitaxe:D8_TEX
Changed lines of the file:
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@@
 			)
 		)
-		(property "Footprint" "Package_SO:SOIC-8_5.3x5.3mm_P1.27mm"
+		(property "Footprint" "bitaxe:D8_TEX"
 			(at 135.128 119.888 0)
 			(hide yes)
@@
 			)
 		)
-		(property "Footprint" "Package_SO:SOIC-8_5.3x5.3mm_P1.27mm"
+		(property "Footprint" "bitaxe:D8_TEX"
 			(at 135.128 89.408 0)
 			(hide yes)
