File: level_shifter.kicad_sch (KiCad schematic)
At the start: 11 parts, among them U19 TLV3542

Commit message: changed fan connector footprint back to normal. lots of part substitutions for JLCPCB. Mounting hole changes for enclosure
Parts:
- C206: DK 490-10700-1-ND -> (none); LCSC C77020 -> C307331; Manufacturer (none) -> Samsung Electro-Mechanics; PARTNO GRM155R71H104KE14D -> CL05B104KB54PNC
- C207: DK 587-5514-1-ND -> (none); Manufacturer (none) -> Samsung Electro-Mechanics; PARTNO EMK105BJ105MV-F -> CL05A105KA5NQNC
- R55, R58, R68, R69: DK 311-1.00KLRCT-ND -> (none); LCSC (none) -> C11702; Manufacturer (none) -> UNI-ROYAL(Uniroyal Elec); PARTNO RC0402FR-071KL -> 0402WGF1001TCE
- R56, R57, R59, R60: DK 311-10KJRCT-ND -> (none); Manufacturer (none) -> UNI-ROYAL(Uniroyal Elec); PARTNO RC0402JR-0710KL -> 0402WGF1002TCE
- U19: value TLV3542 -> OPA2365AIDR; DK 296-45063-1-ND -> (none); LCSC (none) -> C130011; PARTNO TLV3542IDR -> OPA2365AIDR
Other:
- note added: "1V2-0"
- note added: "GND"
- note added: "GND0"

Commit message: updated part attributes for JLCPCB Fabrication Toolkit
Parts:
- U19: FT Rotation Offset (none) -> -90
Changed lines of the file:
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@@
+			)
+		)
+		(property "FT Rotation Offset" "-90"
+			(at 129.54 91.44 0)
+			(hide yes)
+			(show_name no)
+			(do_not_autoplace no)
+			(effects
+				(font
+					(size 1.27 1.27)
+				)
 			)
 		)
@@
 			(at 129.54 60.96 0)
 			(hide yes)
+			(show_name no)
+			(do_not_autoplace no)
+			(effects
+				(font
+					(size 1.27 1.27)
+				)
+			)
+		)
+		(property "FT Rotation Offset" "-90"
+			(at 129.54 60.96 0)
+			(hide yes)
