File: Supply.kicad_sch (KiCad schematic)
At the start: 6 parts, among them J1 XT30, U8 NCS21671SQ050T2G

Commit message: switch to cheaper USB-C connector
Parts:
- J1: PARTNO XT30PW-M -> XT30PW-M30.G.Y
Changed lines of the file:
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@@
 			)
 		)
-		(property "PARTNO" "XT30PW-M"
+		(property "PARTNO" "XT30PW-M30.G.Y"
 			(at 75.946 120.142 0)
 			(effects
